File: Hexapod_Robot_Board.kicad_pcb (KiCad board)
At the start: 4 copper layers, 110 x 90 mm, 105 parts, among them J1 USB-C, SW1 RESET, SW2 BOOT, U1 ESP32-S3-WROOM-1U, U2 BQ25886, U3_L XL4015, U3_R XL4015, U4 AMS1117-3.3, U5 PCA9685_1, U6 PCA9685_2, U7 MPU-6050

Commit message: feat(rev3): Rev 3.0 — Dual ESP32-S3, Vision Coprocessor, BQ25886 charger, triple USB-C, ToF + Camera subsystem
Major architectural upgrade from Rev 2.0:
- Add Vision Coprocessor (ESP32-S3-WROOM-1U-N8R8, U8) — Zephyr esp32s3_eye compatible
- Replace TP5100 with BQ25886 2S LiPo fast charger (PowerPath, USB BC1.2, I2C status)
- Triple South-edge USB-C: J_CHG (dedicated charger), J2 (Main MCU JTAG), J3 (Vision JTAG/video)
- Add 24-pin DVP FPC camera interface (OV3660/OV2640, J_CAM) at top-centre
- Add MaixSense A010 3D ToF (J_TOF) on isolated +5V_TOF linear rail (AMS1117-5.0)
- Add dedicated Vision 3.3V LDO (U_LDO_VIS, AMS1117-3.3) for +3V3_VIS rail
- Add 1-3W camera LED driver (AO3400A Q_CAM_LED, Vision GPIO3)
- Add inter-MCU full-duplex UART link (U1 GPIO43/44 <-> U8 GPIO43/44) + Frame Sync IRQ
- Add external power switch header (J_SW_EXT, 2-pin)
- Add WS2812B-2020 NeoPixel status LED (LED_RGB_MAIN, Main GPIO48)
- Add buzzer (BZ1, R_BZ) for audio alerts
- Schematic annotation confirmed (all semantic refs, 0 unannotated)
- PCB synced from schematic: 3 footprints added (BZ1, C_VBUS_VIS, SW_VIS_RST)
- 98 nets, 528 pads assigned
- Add 3D models: WS2812B-2020, Hirose FH12-24S DVP connector
- Update README to Rev 3.0 with full GPIO tables, power tree, architecture diagram
- Update .gitignore: exclude backups, temp files, __pycache__
Parts:
- added BZ1: Buzzer_Magnetic_3V, Buzzer_Beeper:MagneticBuzzer_Kingstate_KCG0601, F.Cu at (0.00, 0.00)
- added C_CAM1: 10uF, Capacitor_SMD:C_0805_2012Metric, F.Cu at (66.5, -14.0)
- added C_CAM2: 100nF, Capacitor_SMD:C_0603_1608Metric, F.Cu at (66.5, -6.00)
- added C_NEO: 100nF, Capacitor_SMD:C_0603_1608Metric, F.Cu at (75.0, -5.50)
- added C_TOF_IN: 10uF, Capacitor_SMD:C_0805_2012Metric, F.Cu at (48.0, 20.0)
- added C_TOF_OUT: 22uF, Capacitor_SMD:C_0805_2012Metric, F.Cu at (62.0, 20.0)
- added C_U8_1: 10uF, Capacitor_SMD:C_0805_2012Metric, F.Cu at (9.50, -7.00)
- added C_U8_2: 100nF, Capacitor_SMD:C_0603_1608Metric, F.Cu at (9.50, -4.50)
- added C_VBUS_MAIN: 100nF, Capacitor_SMD:C_0603_1608Metric, F.Cu at (105.0, 78.0)
- added C_VBUS_VIS: 100nF, Capacitor_SMD:C_0603_1608Metric, F.Cu at (0.00, 0.00)
- added C_VIS_EN: 1uF, Capacitor_SMD:C_0603_1608Metric, F.Cu at (9.50, -2.50)
- added C_VIS_IN: 10uF, Capacitor_SMD:C_0805_2012Metric, F.Cu at (35.0, 12.0)
- added C_VIS_OUT: 22uF, Capacitor_SMD:C_0805_2012Metric, F.Cu at (48.5, 12.0)
- added D_CAM_LED: SS14, Diode_SMD:D_SOD-123, F.Cu at (42.0, -4.00)
- added J2: USB-C_MAIN, Connector_USB:USB_C_Receptacle_HCTL_HC-TYPE-C-16P-01A, F.Cu at (95.5, 86.1)
- added J3: USB-C_VISION, Connector_USB:USB_C_Receptacle_HCTL_HC-TYPE-C-16P-01A, F.Cu at (84.0, 86.1)
- added J_CAM: OV3660_DVP_24P, Connector_FFC-FPC:Hirose_FH12-24S-0.5SH_1x24-1MP_P0.50mm_Horizontal, F.Cu at (55.0, -7.00)
- added J_CAM_LED: LED_CAM_5V_1-3W, Connector_PinHeader_2.54mm:PinHeader_1x02_P2.54mm_Vertical, F.Cu at (44.0, -11.0)
- added J_SW_EXT: SW_EXT, Connector_PinHeader_2.54mm:PinHeader_1x02_P2.54mm_Vertical, F.Cu at (57.0, 74.0)
- added J_TOF: MaixSense_A010, Connector_PinHeader_2.54mm:PinHeader_1x04_P2.54mm_Vertical, F.Cu at (5.00, -11.0)
- added LED_RGB_MAIN: WS2812B-2020, LED_SMD:LED_WS2812B-2020_PLCC4_2.0x2.0mm, F.Cu at (73.0, -11.0)
- added Q_CAM_LED: AO3400A, Package_TO_SOT_SMD:SOT-23, F.Cu at (36.0, -11.0)
- added R_CAM_LED: 100, Resistor_SMD:R_0603_1608Metric, F.Cu at (36.0, -7.00)
- added R_CAM_SCL: 4.7k, Resistor_SMD:R_0603_1608Metric, F.Cu at (66.5, -8.50)
- added R_CAM_SDA: 4.7k, Resistor_SMD:R_0603_1608Metric, F.Cu at (66.5, -12.0)
- added R_CC3: 5.1k, Resistor_SMD:R_0603_1608Metric, F.Cu at (105.0, 73.0)
- added R_CC4: 5.1k, Resistor_SMD:R_0603_1608Metric, F.Cu at (105.0, 75.5)
- added R_NEO: 330, Resistor_SMD:R_0603_1608Metric, F.Cu at (75.0, -8.00)
- added R_PD_CAM_LED: 10k, Resistor_SMD:R_0603_1608Metric, F.Cu at (36.0, -4.50)
- added R_VIS_BOOT: 10k, Resistor_SMD:R_0603_1608Metric, F.Cu at (36.0, 5.00)
- added R_VIS_CC1: 5.1k, Resistor_SMD:R_0603_1608Metric, F.Cu at (76.5, 85.0)
- added R_VIS_CC2: 5.1k, Resistor_SMD:R_0603_1608Metric, F.Cu at (76.5, 87.5)
- added R_VIS_EN: 10k, Resistor_SMD:R_0603_1608Metric, F.Cu at (9.50, -0.50)
- added SW_VIS_BOOT: SW_Push, Button_Switch_SMD:SW_Push_SPST_NO_Alps_SKRK, F.Cu at (36.0, 1.00)
- added SW_VIS_RST: SW_Push, Button_Switch_SMD:SW_Push_SPST_NO_Alps_SKRK, F.Cu at (0.00, 0.00)
- added U8: ESP32-S3-WROOM-1U-N8R8, RF_Module:ESP32-S3-WROOM-1U, F.Cu at (22.0, 2.50)
- added U_LDO_VIS: AMS1117-3.3, Package_TO_SOT_SMD:SOT-223-3_TabPin2, F.Cu at (42.0, 12.0)
- added U_REG_5V_TOF: AMS1117-5.0, Package_TO_SOT_SMD:SOT-223-3_TabPin2, F.Cu at (55.0, 20.0)
- moved J_BAT 59.8 mm to (14.0, 70.0), turned to 90 degrees
- moved C2 36.7 mm to (74.0, -0.50)
- moved C1 36.2 mm to (74.0, -3.00)
- moved C_ISO2 35.5 mm to (55.0, -2.00)
- moved U1 34.2 mm to (88.0, 2.50)
- moved R1 31.7 mm to (74.0, 2.00)
- moved C3 31.0 mm to (74.0, 4.50)
- moved SW1 29.7 mm to (67.0, -1.00)
- moved D_ISO 29.5 mm to (50.0, -2.00), turned to 0 degrees
- moved C_ISO1 28.0 mm to (53.0, 3.50)
- moved LED_3V3 19.5 mm to (79.0, 20.0)
- moved R_3V3_LED 18.9 mm to (79.0, 22.5)
- moved C_DIV 16.3 mm to (53.0, 14.5), turned to 0 degrees
- moved R_DIV2 16.0 mm to (53.0, 12.0), turned to 0 degrees
- moved R_DIV1 15.7 mm to (53.0, 9.50), turned to 0 degrees
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Connections:
- R_BZ pad 2: GND -> Net-(BZ1-Pad1)
- R_DIV1 pad 2: VBAT_SENSE -> Net-(R_DIV1-Pad2)
- R_DIV2 pad 1: VBAT_SENSE -> Net-(R_DIV1-Pad2)
- SW_PWR pad 2: VBAT_SW -> Net-(SW_PWR-Pad2)
- SW_PWR pad 3: VBAT_SW -> Net-(SW_PWR-Pad2)
- U1 pad 22: unconnected-(U1-IO14-Pad22) -> VISION_RESET
- U1 pad 25: unconnected-(U1-IO48-Pad25) -> Net-(R_NEO-Pad1)
- U1 pad 4: unconnected-(U1-IO4-Pad4) -> VISION_SYNC
- U1 pad 8: unconnected-(U1-IO15-Pad8) -> INTER_UART_RX
- U1 pad 9: unconnected-(U1-IO16-Pad9) -> INTER_UART_TX
- U6 pad 15: unconnected-(U6-LED8-Pad15) -> PWM_L3_T
- U6 pad 16: unconnected-(U6-LED9-Pad16) -> PWM_AUX1
- U6 pad 17: unconnected-(U6-LED10-Pad17) -> PWM_AUX2
- U6 pad 18: unconnected-(U6-LED11-Pad18) -> PWM_AUX3
Routing:
- net VIS_USB_D-: track 0.00 -> 119.5 mm, vias 0 -> 2
- net +3V3_VIS: track 0.00 -> 112.6 mm, vias 0 -> 6
- net VIS_USB_D+: track 0.00 -> 111.8 mm, vias 0 -> 2
- net PWM_3: track 110.1 -> 0.00 mm, vias 2 -> 0
- net PWM_2: track 107.7 -> 0.00 mm, vias 2 -> 0
- net PWM_0: track 102.7 -> 0.00 mm, vias 2 -> 0
- net PWM_1: track 99.0 -> 0.00 mm, vias 2 -> 0
- net PWM_4: track 96.9 -> 0.00 mm, vias 1 -> 0
- net PWM_5: track 94.1 -> 0.00 mm, vias 1 -> 0
- net VISION_RESET: track 0.00 -> 93.2 mm, vias 0 -> 3
- net PWM_6: track 81.8 -> 0.00 mm, vias 1 -> 0
- net PWM_7: track 78.4 -> 0.00 mm, vias 1 -> 0
- net CAM_SDA: track 0.00 -> 78.0 mm
- net PWM_17: track 75.0 -> 0.00 mm, vias 1 -> 0
- net PWM_21: track 75.0 -> 0.00 mm, vias 1 -> 0
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Other:
- board size 110 x 90 mm -> 110 x 106.5 mm
- board text added: "3.3V MAIN"
- board text added: "3.3V VIS"
- board text added: "5V TOF REG"
- board text added: "CAM LED"
- board text added: "CAMERA DVP"
- board text added: "DUAL ESP32-S3 * VISION COPROCESSOR * 3x TYPE-C"
- board text added: "ESP32-S3 MAIN"
- board text added: "ESP32-S3 VIS"
- board text added: "EXT SW"
- board text added: "HEXAPOD ROBOT CONTROLLER REV 3.0"
- board text added: "PWR SW"
- board text added: "RGB STAT"
- board text added: "TOF DEPTH"
- board text added: "USB CHG"
- board text added: "USB MAIN"
- board text added: "USB VISION"
- board text removed: "ESP32-S3-WROOM-1U * MPU-6050 * DUAL 5A BUCK"
- board text removed: "HEXAPOD ROBOT CONTROLLER"
- board text removed: "PWR SWITCH"
- board text removed: "TYPE-C CHG"

Commit message: servo pwm alignments. repo & schematic cleanup
Parts:
- removed H1, H2, H3, H4: M3, MountingHole_3.2mm_M3_Pad_Via
- C1, C_3V3_1, C_PCA2, C_PCA4, C_VBUS1: footprint C_0805_2012Metric -> Capacitor_SMD:C_0805_2012Metric
- C2, C3, C_PCA1, C_PCA3: footprint C_0603_1608Metric -> Capacitor_SMD:C_0603_1608Metric
- C_BAT1: value 22uF -> 22uF_25V; footprint C_1206_3216Metric -> Capacitor_SMD:C_1206_3216Metric
- C_DIV1: renamed from C_DIV; footprint C_0603_1608Metric -> Capacitor_SMD:C_0603_1608Metric
- C_ISO1: footprint CP_Radial_D8.0mm_P3.50mm -> Capacitor_THT:CP_Radial_D8.0mm_P3.50mm
- D_ISO1: renamed from D_ISO; footprint D_SOD-123 -> Diode_SMD:D_SOD-123
- D_STAT1: renamed from D_STAT; footprint LED_0603_1608Metric -> LED_SMD:LED_0603_1608Metric
- J1: footprint USB_C_Receptacle_HCTL_HC-TYPE-C-16P-01A -> Connector_USB:USB_C_Receptacle_HCTL_HC-TYPE-C-16P-01A
- J_AUX1: value AUX_1 -> AUX_R_9; footprint PinHeader_1x03_P2.54mm_Vertical -> Connector_PinHeader_2.54mm:PinHeader_1x03_P2.54mm_Vertical
- J_AUX2: value AUX_2 -> AUX_R_10; footprint PinHeader_1x03_P2.54mm_Vertical -> Connector_PinHeader_2.54mm:PinHeader_1x03_P2.54mm_Vertical
- J_AUX3: value AUX_3 -> AUX_R_11; footprint PinHeader_1x03_P2.54mm_Vertical -> Connector_PinHeader_2.54mm:PinHeader_1x03_P2.54mm_Vertical
- J_AUX4: value AUX_4 -> AUX_L_9; footprint PinHeader_1x03_P2.54mm_Vertical -> Connector_PinHeader_2.54mm:PinHeader_1x03_P2.54mm_Vertical
- J_AUX5: value AUX_5 -> AUX_L_10; footprint PinHeader_1x03_P2.54mm_Vertical -> Connector_PinHeader_2.54mm:PinHeader_1x03_P2.54mm_Vertical
- J_AUX6: value AUX_6 -> AUX_L_11; footprint PinHeader_1x03_P2.54mm_Vertical -> Connector_PinHeader_2.54mm:PinHeader_1x03_P2.54mm_Vertical
- J_BAT1: renamed from J_BAT; value 2S_LiPo -> 2S_LiPo_7.4V; footprint AMASS_XT30PW-M_1x02_P2.50mm_Horizontal -> Connector_AMASS:AMASS_XT30PW-M_1x02_P2.50mm_Horizontal
- J_I2C1: renamed from J_I2C; footprint PinHeader_1x04_P2.54mm_Vertical -> Connector_PinHeader_2.54mm:PinHeader_1x04_P2.54mm_Vertical
- J_L1_C1: renamed from J_L1_C; footprint PinHeader_1x03_P2.54mm_Vertical -> Connector_PinHeader_2.54mm:PinHeader_1x03_P2.54mm_Vertical
- J_L1_F1: renamed from J_L1_F; footprint PinHeader_1x03_P2.54mm_Vertical -> Connector_PinHeader_2.54mm:PinHeader_1x03_P2.54mm_Vertical
- J_L1_T1: renamed from J_L1_T; footprint PinHeader_1x03_P2.54mm_Vertical -> Connector_PinHeader_2.54mm:PinHeader_1x03_P2.54mm_Vertical
- J_L2_C1: renamed from J_L2_C; footprint PinHeader_1x03_P2.54mm_Vertical -> Connector_PinHeader_2.54mm:PinHeader_1x03_P2.54mm_Vertical
- J_L2_F1: renamed from J_L2_F; footprint PinHeader_1x03_P2.54mm_Vertical -> Connector_PinHeader_2.54mm:PinHeader_1x03_P2.54mm_Vertical
- J_L2_T1: renamed from J_L2_T; footprint PinHeader_1x03_P2.54mm_Vertical -> Connector_PinHeader_2.54mm:PinHeader_1x03_P2.54mm_Vertical
- J_L3_C1: renamed from J_L3_C; footprint PinHeader_1x03_P2.54mm_Vertical -> Connector_PinHeader_2.54mm:PinHeader_1x03_P2.54mm_Vertical
- J_L3_F1: renamed from J_L3_F; footprint PinHeader_1x03_P2.54mm_Vertical -> Connector_PinHeader_2.54mm:PinHeader_1x03_P2.54mm_Vertical
- J_L3_T1: renamed from J_L3_T; footprint PinHeader_1x03_P2.54mm_Vertical -> Connector_PinHeader_2.54mm:PinHeader_1x03_P2.54mm_Vertical
- J_L4_C1: renamed from J_L4_C; footprint PinHeader_1x03_P2.54mm_Vertical -> Connector_PinHeader_2.54mm:PinHeader_1x03_P2.54mm_Vertical
- J_L4_F1: renamed from J_L4_F; footprint PinHeader_1x03_P2.54mm_Vertical -> Connector_PinHeader_2.54mm:PinHeader_1x03_P2.54mm_Vertical
- J_L4_T1: renamed from J_L4_T; footprint PinHeader_1x03_P2.54mm_Vertical -> Connector_PinHeader_2.54mm:PinHeader_1x03_P2.54mm_Vertical
- J_L5_C1: renamed from J_L5_C; footprint PinHeader_1x03_P2.54mm_Vertical -> Connector_PinHeader_2.54mm:PinHeader_1x03_P2.54mm_Vertical
- J_L5_F1: renamed from J_L5_F; footprint PinHeader_1x03_P2.54mm_Vertical -> Connector_PinHeader_2.54mm:PinHeader_1x03_P2.54mm_Vertical
- J_L5_T1: renamed from J_L5_T; footprint PinHeader_1x03_P2.54mm_Vertical -> Connector_PinHeader_2.54mm:PinHeader_1x03_P2.54mm_Vertical
- J_L6_C1: renamed from J_L6_C; footprint PinHeader_1x03_P2.54mm_Vertical -> Connector_PinHeader_2.54mm:PinHeader_1x03_P2.54mm_Vertical
- J_L6_F1: renamed from J_L6_F; footprint PinHeader_1x03_P2.54mm_Vertical -> Connector_PinHeader_2.54mm:PinHeader_1x03_P2.54mm_Vertical
- J_L6_T1: renamed from J_L6_T; footprint PinHeader_1x03_P2.54mm_Vertical -> Connector_PinHeader_2.54mm:PinHeader_1x03_P2.54mm_Vertical
- J_SW_EXT1: renamed from J_SW_EXT; value SW_EXT -> EXT_SW
- J_UART1: renamed from J_UART; footprint PinHeader_1x04_P2.54mm_Vertical -> Connector_PinHeader_2.54mm:PinHeader_1x04_P2.54mm_Vertical
- LED_3V3: footprint LED_0603_1608Metric -> LED_SMD:LED_0603_1608Metric
- LED_CHG1: renamed from LED_CHG; footprint LED_0603_1608Metric -> LED_SMD:LED_0603_1608Metric
- LED_FULL1: renamed from LED_FULL; footprint LED_0603_1608Metric -> LED_SMD:LED_0603_1608Metric
- L_CHG1: renamed from L_CHG; footprint L_7.3x7.3_H4.5 -> Inductor_SMD:L_7.3x7.3_H4.5
- R1, R2, R_DIV1, R_DIV2: footprint R_0603_1608Metric -> Resistor_SMD:R_0603_1608Metric
- R_CC1, R_CC2: value 5.1k -> 5.1k_1%; footprint R_0603_1608Metric -> Resistor_SMD:R_0603_1608Metric
- R_OE1: renamed from R_OE; footprint R_0603_1608Metric -> Resistor_SMD:R_0603_1608Metric
- R_SCL1: renamed from R_SCL; footprint R_0603_1608Metric -> Resistor_SMD:R_0603_1608Metric
- R_SDA1: renamed from R_SDA; footprint R_0603_1608Metric -> Resistor_SMD:R_0603_1608Metric
- R_STAT1: renamed from R_STAT; footprint R_0603_1608Metric -> Resistor_SMD:R_0603_1608Metric
- SW1, SW2: footprint SW_Push_SPST_NO_Alps_SKRK -> Button_Switch_SMD:SW_Push_SPST_NO_Alps_SKRK
- SW_PWR1: renamed from SW_PWR; value POWER -> PWR_SW; footprint SW_Slide_SPDT_Straight_CK_OS102011MS2Q -> Button_Switch_THT:SW_Slide_SPDT_Straight_CK_OS102011MS2Q
- U1: footprint ESP32-S3-WROOM-1U -> RF_Module:ESP32-S3-WROOM-1U
- U2: footprint QFN-24-1EP_4x4mm_P0.5mm_EP2.7x2.7mm_ThermalVias -> Package_DFN_QFN:QFN-24-1EP_4x4mm_P0.5mm_EP2.7x2.7mm_ThermalVias
- U4: footprint SOT-223-3_TabPin2 -> Package_TO_SOT_SMD:SOT-223-3_TabPin2
- U5: value PCA9685_1 -> PCA9685_0x40; footprint TSSOP-28_4.4x9.7mm_P0.65mm -> Package_SO:TSSOP-28_4.4x9.7mm_P0.65mm
- U6: value PCA9685_2 -> PCA9685_0x41; footprint TSSOP-28_4.4x9.7mm_P0.65mm -> Package_SO:TSSOP-28_4.4x9.7mm_P0.65mm
- moved BZ1 88.3 mm to (56.9, 67.5)
- moved U6 58.4 mm to (25.9, 67.0)
- moved U5 58.1 mm to (83.9, 61.9)
- moved C_VBUS_VIS1 40.6 mm to (40.0, -7.00)
- moved SW_VIS_RST1 23.8 mm to (20.5, -12.0)
- renumbered C_IN1_L to C_IN1_L1, C_IN1_R to C_IN1_R1, C_IN2_L to C_IN2_L1, C_IN2_R to C_IN2_R1, C_NEO to C_NEO1, C_OUT1_L to C_OUT1_L1, C_OUT1_R to C_OUT1_R1, C_OUT2_L to C_OUT2_L1, C_OUT2_R to C_OUT2_R1, C_OUT3_L to C_OUT3_L1, C_OUT3_R to C_OUT3_R1, C_TOF_IN to C_TOF_IN1, C_TOF_OUT to C_TOF_OUT1, C_VBUS_MAIN to C_VBUS_MAIN1, C_VBUS_VIS to C_VBUS_VIS1, C_VIS_EN to C_VIS_EN1, C_VIS_IN to C_VIS_IN1, C_VIS_OUT to C_VIS_OUT1, D_CAM_LED to D_CAM_LED1, D_CATCH_L to D_CATCH_L1, D_CATCH_R to D_CATCH_R1, J_CAM to J_CAM1, J_CAM_LED to J_CAM_LED1, J_TOF to J_TOF1, LED_L to LED_L1, LED_R to LED_R1, LED_RGB_MAIN to LED_RGB_MAIN1, L_SERVO_L to L_SERVO_L1, L_SERVO_R to L_SERVO_R1, Q_CAM_LED to Q_CAM_LED1, R_3V3_LED to R_3V3_LED1, R_BZ to R_BZ1, R_CAM_LED to R_CAM_LED1, R_CAM_SCL to R_CAM_SCL1, R_CAM_SDA to R_CAM_SDA1, R_CHG to R_CHG1, R_FB1_L to R_FB1_L1, R_FB1_R to R_FB1_R1, R_FB2_L to R_FB2_L1, R_FB2_R to R_FB2_R1, R_FULL to R_FULL1, R_LED_L to R_LED_L1, R_LED_R to R_LED_R1, R_NEO to R_NEO1, R_PD_CAM_LED to R_PD_CAM_LED1, R_VIS_BOOT to R_VIS_BOOT1, R_VIS_EN to R_VIS_EN1, SW_VIS_BOOT to SW_VIS_BOOT1, SW_VIS_RST to SW_VIS_RST1, U3_L to U3_L1, U3_R to U3_R1, U_LDO_VIS to U_LDO_VIS1, U_REG_5V_TOF to U_REG_5V_TOF1
Connections:
- net BUCK_SW_L renamed Net-(D_CATCH_L1-A)
- net BUCK_SW_R renamed Net-(D_CATCH_R1-A)
- net PWM_0 renamed PWM_R_0
- net PWM_1 renamed PWM_R_1
- net PWM_2 renamed PWM_R_2
- net PWM_3 renamed PWM_R_3
- net PWM_4 renamed PWM_R_4
- net PWM_5 renamed PWM_R_5
- net PWM_6 renamed PWM_R_6
- net PWM_7 renamed PWM_R_7
- net PWM_8 renamed PWM_R_8
- C_VBUS_MAIN1 pad 2: GND -> VBUS_MAIN
- C_VBUS_VIS1 pad 2: (no net) -> VBUS_VIS
- J2 pad A8: (no net) -> unconnected-(J2-SBU1-PadA8)
- J2 pad B8: (no net) -> unconnected-(J2-SBU2-PadB8)
- J3 pad A8: (no net) -> unconnected-(J3-SBU1-PadA8)
- J3 pad B8: (no net) -> unconnected-(J3-SBU2-PadB8)
- J_AUX1 pad 3: PWM_18 -> PWM_R_9
- J_AUX2 pad 3: PWM_19 -> PWM_R_10
- J_AUX3 pad 3: PWM_20 -> PWM_R_11
- J_AUX4 pad 3: PWM_21 -> PWM_L_9
- J_AUX5 pad 3: PWM_22 -> PWM_L_10
- J_AUX6 pad 3: PWM_23 -> PWM_L_11
- J_CAM1 pad 1: (no net) -> unconnected-(J_CAM1-Pin_1-Pad1)
- J_L4_C1 pad 3: PWM_9 -> PWM_L_0
- J_L4_F1 pad 3: PWM_10 -> PWM_L_1
- J_L4_T1 pad 3: PWM_11 -> PWM_L_2
- J_L5_C1 pad 3: PWM_12 -> PWM_L_3
- J_L5_F1 pad 3: PWM_13 -> PWM_L_4
- J_L5_T1 pad 3: PWM_14 -> PWM_L_5
- J_L6_C1 pad 3: PWM_15 -> PWM_L_6
- J_L6_F1 pad 3: PWM_16 -> PWM_L_7
- J_L6_T1 pad 3: PWM_17 -> PWM_L_8
- LED_3V3 pad 2: GND -> Net-(LED_3V3-A)
- LED_RGB_MAIN1 pad 1: (no net) -> unconnected-(LED_RGB_MAIN1-DOUT-Pad1)
- R_3V3_LED1 pad 1: +3V3 -> Net-(LED_3V3-A)
- R_DIV1 pad 2: Net-(R_DIV1-Pad2) -> VBAT_SENSE
- R_DIV2 pad 1: Net-(R_DIV1-Pad2) -> VBAT_SENSE
- R_FB1_L1 pad 1: V_SERVO_L -> Net-(U3_L1-FB)
- R_FB1_L1 pad 2: BUCK_FB_L -> V_SERVO_L
- R_FB1_R1 pad 1: V_SERVO_R -> Net-(U3_R1-FB)
- R_FB1_R1 pad 2: BUCK_FB_R -> V_SERVO_R
- R_FB2_L1 pad 1: BUCK_FB_L -> Net-(U3_L1-FB)
- R_FB2_R1 pad 1: BUCK_FB_R -> Net-(U3_R1-FB)
- SW_PWR1 pad 2: Net-(SW_PWR-Pad2) -> VBAT_SW
- SW_PWR1 pad 3: Net-(SW_PWR-Pad2) -> VBAT_SW
- U1 pad : GND -> (no net)
- U2 pad : GND -> (no net)
- U2 pad 15: unconnected-(U2-SYS-Pad15) -> unconnected-(U2-SYS-Pad15)_1
- U3_L1 pad 2: BUCK_FB_L -> Net-(U3_L1-FB)
- U3_R1 pad 2: BUCK_FB_R -> Net-(U3_R1-FB)
- U5 pad 16: PWM_9 -> PWM_R_9
- U5 pad 17: PWM_10 -> PWM_R_10
- U5 pad 18: PWM_11 -> PWM_R_11
- U5 pad 19: PWM_12 -> unconnected-(U5-LED12-Pad19)
- U5 pad 20: PWM_13 -> unconnected-(U5-LED13-Pad20)
- U5 pad 21: PWM_14 -> unconnected-(U5-LED14-Pad21)
- U5 pad 22: PWM_15 -> unconnected-(U5-LED15-Pad22)
- U6 pad 10: PWM_20 -> PWM_L_4
- U6 pad 11: PWM_21 -> PWM_L_5
- U6 pad 12: PWM_22 -> PWM_L_6
- U6 pad 13: PWM_23 -> PWM_L_7
- U6 pad 15: PWM_L3_T -> PWM_L_8
- U6 pad 16: PWM_AUX1 -> PWM_L_9
- U6 pad 17: PWM_AUX2 -> PWM_L_10
- U6 pad 18: PWM_AUX3 -> PWM_L_11
- U6 pad 6: PWM_16 -> PWM_L_0
- U6 pad 7: PWM_17 -> PWM_L_1
- U6 pad 8: PWM_18 -> PWM_L_2
- U6 pad 9: PWM_19 -> PWM_L_3
- U8 pad 16: (no net) -> unconnected-(U8-IO46-Pad16)
- U8 pad 22: (no net) -> unconnected-(U8-IO14-Pad22)
- U8 pad 25: (no net) -> unconnected-(U8-IO48-Pad25)
- U8 pad 26: (no net) -> unconnected-(U8-IO45-Pad26)
- U8 pad 28: (no net) -> unconnected-(U8-IO35-Pad28)
- U8 pad 29: (no net) -> unconnected-(U8-IO36-Pad29)
- U8 pad 30: (no net) -> unconnected-(U8-IO37-Pad30)
- U8 pad 31: (no net) -> unconnected-(U8-IO38-Pad31)
- U8 pad 32: (no net) -> unconnected-(U8-IO39-Pad32)
- U8 pad 33: (no net) -> unconnected-(U8-IO40-Pad33)
- U8 pad 34: (no net) -> unconnected-(U8-IO41-Pad34)
- U8 pad 35: (no net) -> unconnected-(U8-IO42-Pad35)
Routing:
- net PWM_L_0: track 0.00 -> 59.1 mm, vias 0 -> 1
- net PWM_L4_C: track 59.1 -> 0.00 mm, vias 1 -> 0
- net PWM_R_0: track 0.00 -> 56.5 mm, vias 0 -> 1
- net PWM_L1_C: track 56.5 -> 0.00 mm, vias 1 -> 0
- net PWM_L_1: track 0.00 -> 52.9 mm, vias 0 -> 1
- net PWM_L4_F: track 52.9 -> 0.00 mm, vias 1 -> 0
- net PWM_R_1: track 0.00 -> 50.1 mm, vias 0 -> 1
- net PWM_L1_F: track 50.1 -> 0.00 mm, vias 1 -> 0
- net PWM_L_2: track 0.00 -> 48.6 mm, vias 0 -> 1
- net PWM_L4_T: track 48.6 -> 0.00 mm, vias 1 -> 0
- net PWM_R_2: track 0.00 -> 46.2 mm, vias 0 -> 2
- net PWM_L1_T: track 46.2 -> 0.00 mm, vias 2 -> 0
- net PWM_L_3: track 0.00 -> 40.5 mm, vias 0 -> 1
- net PWM_L5_C: track 40.5 -> 0.00 mm, vias 1 -> 0
- net PWM_R_3: track 0.00 -> 38.8 mm, vias 0 -> 1
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