File: Hexapod_Robot_Board.kicad_sch (KiCad schematic)
At the start: 84 parts, among them J1 USB-C, SW1 RESET, SW2 BOOT, U1 ESP32-S3-WROOM-1, U2 BQ25886, U3 XL4015, U4 AMS1117-3.3, U5 PCA9685_0x40, U6 PCA9685_0x41

Commit message: Enhance schematic design: 7 clean functional blocks, physical wire traces, and 0-ERC validation
Connections:
- no-connect marks 48 -> 46
Other:
- note added: "3-Pin Headers (GND, 5V, PWM): Legs 1-6 (Coxa, Femur, Tibia) + 6 AUX PWM"
- note added: "AMS1117-3.3 Low-Noise Supply for ESP32-S3 and PCA9685 Logic"
- note added: "Dual PCA9685PW 12-Bit PWM Drivers (0x40 & 0x41)"
- note added: "Dual-core 240MHz XTensa, Auto-Reset, Boot, UART & I2C Expansion"
- note added: "SECTION 1: USB TYPE-C & 2S LIPO CHARGER"
- note added: "SECTION 2: BATTERY & TELEMETRY"
- note added: "SECTION 3: 5V/3A SERVO BUCK REGULATOR"
- note added: "SECTION 4: 3.3V SYSTEM LOGIC LDO"
- note added: "SECTION 5: ESP32-S3-WROOM-1 MCU"
- note added: "SECTION 6: DUAL 16-CH PWM CONTROLLERS"
- note added: "SECTION 7: 18-DOF SERVO HEADERS & AUX PWM"
- note added: "TP5100 / BQ25886 8.4V/1.5A Switching Fast Charger with CC Detection"
- note added: "XL4015 High-Current Buck Converter for 18 Hexapod Servos"
- note added: "XT30 2S LiPo Input, Power Switch, Diode & 1% ADC Telemetry Divider"
- moved on the sheet: C1, C2, C3, C_3V3_1, C_3V3_2, C_BAT1, C_BAT2, C_DIV, C_IN1, C_IN2, C_ISO1, C_ISO2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

Commit message: feat(pcb): complete Rev 2.0 4-layer routing, achieve 0 DRC / 0 ERC, and export fabrication package
Parts:
- removed C_IN1: 100uF_25V, Capacitor_THT:CP_Radial_D8.0mm_P3.50mm, symbol Device:C
- removed C_IN2: 22uF_25V, Capacitor_SMD:C_1206_3216Metric, symbol Device:C
- removed C_OUT1: 1000uF_10V, Capacitor_THT:CP_Radial_D8.0mm_P3.50mm, symbol Device:C
- removed C_OUT2: 22uF_16V, Capacitor_SMD:C_1206_3216Metric, symbol Device:C
- removed C_OUT3: 100nF, Capacitor_SMD:C_0603_1608Metric, symbol Device:C
- removed D_CATCH: SS54, Diode_SMD:D_SMC, symbol Device:D_Schottky
- removed LED_SERVO: Green, LED_SMD:LED_0603_1608Metric, symbol Device:LED
- removed L_SERVO: 10uH_10A, Inductor_SMD:L_12x12mm_H8mm, symbol Device:L
- removed R_FB1: 10k_1%, Resistor_SMD:R_0603_1608Metric, symbol Device:R
- removed R_FB2: 3.16k_1%, Resistor_SMD:R_0603_1608Metric, symbol Device:R
- removed R_SERVO_LED: 1k, Resistor_SMD:R_0603_1608Metric, symbol Device:R
- removed U3: XL4015, Package_TO_SOT_SMD:TO-263-5_TabPin3, symbol Regulator_Switching:XL4015
- added C_IN1_L, C_IN1_R: 100uF_25V, Capacitor_THT:CP_Radial_D8.0mm_P3.50mm, symbol Device:C
- added C_IN2_L, C_IN2_R: 22uF_25V, Capacitor_SMD:C_1206_3216Metric, symbol Device:C
- added C_MPU1, C_MPU2, C_MPU3, C_OUT3_L, C_OUT3_R: 100nF, Capacitor_SMD:C_0603_1608Metric, symbol Device:C
- added C_MPU5: 2.2nF, Capacitor_SMD:C_0603_1608Metric, symbol Device:C
- added C_OUT1_L, C_OUT1_R: 1000uF_10V, Capacitor_THT:CP_Radial_D8.0mm_P3.50mm, symbol Device:C
- added C_OUT2_L, C_OUT2_R: 22uF_16V, Capacitor_SMD:C_1206_3216Metric, symbol Device:C
- added D_CATCH_L, D_CATCH_R: SS54, Diode_SMD:D_SMC, symbol Device:D_Schottky
- added LED_L, LED_R: Green, LED_SMD:LED_0805_2012Metric, symbol Device:LED
- added L_SERVO_L, L_SERVO_R: 10uH_10A, Inductor_SMD:L_12x12mm_H8mm, symbol Device:L
- added R_FB1_L, R_FB1_R: 10k_1%, Resistor_SMD:R_0603_1608Metric, symbol Device:R
- added R_FB2_L, R_FB2_R: 3.16k_1%, Resistor_SMD:R_0603_1608Metric, symbol Device:R
- added R_LED_L, R_LED_R: 1k, Resistor_SMD:R_0603_1608Metric, symbol Device:R
- added U3_L, U3_R: XL4015, Package_TO_SOT_SMD:TO-263-5_TabPin3, symbol Regulator_Switching:XL4015
- added U7: MPU-6050, Sensor_Motion:InvenSense_QFN-24_4x4mm_P0.5mm, symbol Sensor_Motion:MPU-6050
- U1: value ESP32-S3-WROOM-1 -> ESP32-S3-WROOM-1U; footprint RF_Module:ESP32-S3-WROOM-1 -> RF_Module:ESP32-S3-WROOM-1U
Connections:
- net +3V3: now also C_MPU1.1, C_MPU3.1, U7.13 (VDD), U7.8 (VLOGIC)
- net GND: now also C_IN1_L.2, C_IN1_R.2, C_IN2_L.2, C_IN2_R.2, C_MPU1.2, C_MPU2.2, C_MPU3.2, C_MPU5.2, C_OUT1_L.2, C_OUT1_R.2, C_OUT2_L.2, C_OUT2_R.2, C_OUT3_L.2, C_OUT3_R.2, D_CATCH_L.1 (K), D_CATCH_R.1 (K), R_FB2_L.2, R_FB2_R.2, R_LED_L.2, R_LED_R.2, U3_L.1 (GND), U3_L.4 (VC), U3_R.1 (GND), U3_R.4 (VC), U7.1 (CLKIN), U7.11 (FSYNC), U7.18 (GND), U7.9 (AD0)
- net I2C_SCL: now also U7.23 (SCL)
- net I2C_SDA: now also U7.24 (SDA)
- net VBAT_SW: now also C_IN1_L.1, C_IN1_R.1, C_IN2_L.1, C_IN2_R.1, U3_L.5 (VIN), U3_R.5 (VIN)
- net MPU_INT: now reaches U1.11 (IO18)
- net MPU_INT: now also U7.12 (INT)
- net V_SERVO renamed V_SERVO_L
- net V_SERVO_L: now also C_OUT1_L.1, C_OUT2_L.1, C_OUT3_L.1, LED_L.1 (K), L_SERVO_L.2, R_FB1_L.1; no longer J_AUX1.2 (Pin_2), J_AUX2.2 (Pin_2), J_AUX3.2 (Pin_2), J_L1_C.2 (Pin_2), J_L1_F.2 (Pin_2), J_L1_T.2 (Pin_2), J_L2_C.2 (Pin_2), J_L2_F.2 (Pin_2), J_L2_T.2 (Pin_2), J_L3_C.2 (Pin_2), J_L3_F.2 (Pin_2), J_L3_T.2 (Pin_2)
- new net: C_MPU2.1, U7.10 (REGOUT)
- new net: C_MPU5.1, U7.20 (CPOUT)
- new net: LED_L.2 (A), R_LED_L.1
- new net: LED_R.2 (A), R_LED_R.1
- new net BUCK_FB_L: R_FB1_L.2, R_FB2_L.1, U3_L.2 (FB)
- new net BUCK_FB_R: R_FB1_R.2, R_FB2_R.1, U3_R.2 (FB)
- new net BUCK_SW_L: D_CATCH_L.2 (A), L_SERVO_L.1, U3_L.3 (SW)
- new net BUCK_SW_R: D_CATCH_R.2 (A), L_SERVO_R.1, U3_R.3 (SW)
- new net V_SERVO_R: C_OUT1_R.1, C_OUT2_R.1, C_OUT3_R.1, J_AUX1.2 (Pin_2), J_AUX2.2 (Pin_2), J_AUX3.2 (Pin_2), J_L1_C.2 (Pin_2), J_L1_F.2 (Pin_2), J_L1_T.2 (Pin_2), J_L2_C.2 (Pin_2), J_L2_F.2 (Pin_2), J_L2_T.2 (Pin_2), J_L3_C.2 (Pin_2), J_L3_F.2 (Pin_2), J_L3_T.2 (Pin_2), LED_R.1 (K), L_SERVO_R.2, R_FB1_R.1
- no-connect marks 46 -> 48
Other:
- note added: "Dual XL4015 Converters: V_SERVO_R (Right Servos) & V_SERVO_L (Left Servos)"
- note added: "SECTION 3: DUAL 5V/5A SERVO BUCK REGULATORS (10A TOTAL)"
- note added: "SECTION 3A: RIGHT SERVO BUCK (5V/5A, V_SERVO_R)"
- note added: "SECTION 3B: LEFT SERVO BUCK (5V/5A, V_SERVO_L)"
- note added: "SECTION 8: MPU-6050 6-AXIS MOTION TRACKING SENSOR"
- note removed: "SECTION 3: 5V/3A SERVO BUCK REGULATOR"
- note removed: "XL4015 High-Current Buck Converter for 18 Hexapod Servos"

Commit message: feat(rev3): Rev 3.0 — Dual ESP32-S3, Vision Coprocessor, BQ25886 charger, triple USB-C, ToF + Camera subsystem
Major architectural upgrade from Rev 2.0:
- Add Vision Coprocessor (ESP32-S3-WROOM-1U-N8R8, U8) — Zephyr esp32s3_eye compatible
- Replace TP5100 with BQ25886 2S LiPo fast charger (PowerPath, USB BC1.2, I2C status)
- Triple South-edge USB-C: J_CHG (dedicated charger), J2 (Main MCU JTAG), J3 (Vision JTAG/video)
- Add 24-pin DVP FPC camera interface (OV3660/OV2640, J_CAM) at top-centre
- Add MaixSense A010 3D ToF (J_TOF) on isolated +5V_TOF linear rail (AMS1117-5.0)
- Add dedicated Vision 3.3V LDO (U_LDO_VIS, AMS1117-3.3) for +3V3_VIS rail
- Add 1-3W camera LED driver (AO3400A Q_CAM_LED, Vision GPIO3)
- Add inter-MCU full-duplex UART link (U1 GPIO43/44 <-> U8 GPIO43/44) + Frame Sync IRQ
- Add external power switch header (J_SW_EXT, 2-pin)
- Add WS2812B-2020 NeoPixel status LED (LED_RGB_MAIN, Main GPIO48)
- Add buzzer (BZ1, R_BZ) for audio alerts
- Schematic annotation confirmed (all semantic refs, 0 unannotated)
- PCB synced from schematic: 3 footprints added (BZ1, C_VBUS_VIS, SW_VIS_RST)
- 98 nets, 528 pads assigned
- Add 3D models: WS2812B-2020, Hirose FH12-24S DVP connector
- Update README to Rev 3.0 with full GPIO tables, power tree, architecture diagram
- Update .gitignore: exclude backups, temp files, __pycache__
Parts:
- added BZ1: Buzzer_Magnetic_3V, Buzzer_Beeper:MagneticBuzzer_Kingstate_KCG0601, symbol Device:Buzzer
- added C_CAM1, C_TOF_IN, C_U8_1, C_VIS_IN: 10uF, Capacitor_SMD:C_0805_2012Metric, symbol Device:C
- added C_CAM2, C_NEO, C_U8_2, C_VBUS_MAIN, C_VBUS_VIS: 100nF, Capacitor_SMD:C_0603_1608Metric, symbol Device:C
- added C_TOF_OUT, C_VIS_OUT: 22uF, Capacitor_SMD:C_0805_2012Metric, symbol Device:C
- added C_VIS_EN: 1uF, Capacitor_SMD:C_0603_1608Metric, symbol Device:C
- added D_CAM_LED: SS14, Diode_SMD:D_SOD-123, symbol Device:D_Schottky
- added J2: USB-C_MAIN, Connector_USB:USB_C_Receptacle_HCTL_HC-TYPE-C-16P-01A, symbol Connector:USB_C_Receptacle_USB2.0_16P
- added J3: USB-C_VISION, Connector_USB:USB_C_Receptacle_HCTL_HC-TYPE-C-16P-01A, symbol Connector:USB_C_Receptacle_USB2.0_16P
- added J_CAM: OV3660_DVP_24P, Connector_FFC-FPC:Hirose_FH12-24S-0.5SH_1x24-1MP_P0.50mm_Horizontal, symbol Connector_Generic:Conn_01x24
- added J_CAM_LED: LED_CAM_5V_1-3W, Connector_PinHeader_2.54mm:PinHeader_1x02_P2.54mm_Vertical, symbol Connector_Generic:Conn_01x02
- added J_SW_EXT: SW_EXT, Connector_PinHeader_2.54mm:PinHeader_1x02_P2.54mm_Vertical, symbol Connector_Generic:Conn_01x02
- added J_TOF: MaixSense_A010, Connector_PinHeader_2.54mm:PinHeader_1x04_P2.54mm_Vertical, symbol Connector_Generic:Conn_01x04
- added LED_RGB_MAIN: WS2812B-2020, LED_SMD:LED_WS2812B-2020_PLCC4_2.0x2.0mm, symbol LED:WS2812B-2020
- added Q_CAM_LED: AO3400A, Package_TO_SOT_SMD:SOT-23, symbol Transistor_FET:Q_NMOS_GSD
- added R_CAM_LED: 100, Resistor_SMD:R_0603_1608Metric, symbol Device:R
- added R_CAM_SCL, R_CAM_SDA: 4.7k, Resistor_SMD:R_0603_1608Metric, symbol Device:R
- added R_CC3, R_CC4, R_VIS_CC1, R_VIS_CC2: 5.1k, Resistor_SMD:R_0603_1608Metric, symbol Device:R
- added R_NEO: 330, Resistor_SMD:R_0603_1608Metric, symbol Device:R
- added R_PD_CAM_LED, R_VIS_BOOT, R_VIS_EN: 10k, Resistor_SMD:R_0603_1608Metric, symbol Device:R
- added SW_VIS_BOOT, SW_VIS_RST: SW_Push, Button_Switch_SMD:SW_Push_SPST_NO_Alps_SKRK, symbol Switch:SW_Push
- added U8: ESP32-S3-WROOM-1U-N8R8, RF_Module:ESP32-S3-WROOM-1U, symbol RF_Module:ESP32-S3-WROOM-1
- added U_LDO_VIS: AMS1117-3.3, Package_TO_SOT_SMD:SOT-223-3_TabPin2, symbol Regulator_Linear:AMS1117-3.3
- added U_REG_5V_TOF: AMS1117-5.0, Package_TO_SOT_SMD:SOT-223-3_TabPin2, symbol Regulator_Linear:AMS1117-3.3
Connections:
- net +3V3: now also C_NEO.1, LED_RGB_MAIN.4 (VDD)
- net GND: now also BZ1.2 (-), C_CAM1.2, C_CAM2.2, C_NEO.2, C_TOF_IN.2, C_TOF_OUT.2, C_U8_1.1, C_U8_2.1, C_VBUS_MAIN.1, C_VBUS_VIS.1, C_VIS_EN.1, C_VIS_IN.2, C_VIS_OUT.2, J2.A1 (GND), J2.A12 (GND), J2.B1 (GND), J2.B12 (GND), J2.SH (SHIELD), J3.A1 (GND), J3.A12 (GND), J3.B1 (GND), J3.B12 (GND), J3.SH (SHIELD), J_CAM.15 (Pin_15), J_CAM.2 (Pin_2), J_CAM.23 (Pin_23), J_CAM.24 (Pin_24), J_TOF.2 (Pin_2), LED_RGB_MAIN.2 (VSS), Q_CAM_LED.2 (S), R_CC3.2, R_CC4.2, R_PD_CAM_LED.2, R_VIS_CC1.2, R_VIS_CC2.2, SW_VIS_BOOT.1, SW_VIS_RST.1, U8.1 (GND), U8.40 (GND), U8.41 (GND), U_LDO_VIS.1 (GND), U_REG_5V_TOF.1 (GND); no longer R_BZ.2
- net USB_D+: now also J2.A6 (D+), J2.B6 (D+)
- net USB_D-: now also J2.A7 (D-), J2.B7 (D-)
- net VBAT: now also J_SW_EXT.1 (Pin_1)
- net VBAT_SW: now also C_TOF_IN.1, C_VIS_IN.1, J_SW_EXT.2 (Pin_2), U_LDO_VIS.3 (VI), U_REG_5V_TOF.3 (VI)
- net VISION_RESET: now reaches U1.22 (IO14)
- net VISION_RESET: now also C_VIS_EN.2, R_VIS_EN.2, SW_VIS_RST.2, U8.3 (EN)
- net at U1.25 (IO48): now also R_NEO.1
- net VISION_SYNC: now reaches U1.4 (IO4)
- net VISION_SYNC: now also U8.23 (IO21)
- net INTER_UART_RX: now reaches U1.8 (IO15)
- net INTER_UART_RX: now also U8.36 (RXD0)
- net INTER_UART_TX: now reaches U1.9 (IO16)
- net INTER_UART_TX: now also U8.37 (TXD0)
- new net: BZ1.1 (+), R_BZ.2
- new net: J2.A5 (CC1), R_CC3.1
- new net: Q_CAM_LED.1 (G), R_CAM_LED.2, R_PD_CAM_LED.1
- new net: J3.A5 (CC1), R_VIS_CC1.1
- new net: J2.B5 (CC2), R_CC4.1
- new net: LED_RGB_MAIN.3 (DIN), R_NEO.2
- new net: J3.B5 (CC2), R_VIS_CC2.1
- new net +3V3_VIS: C_CAM1.1, C_CAM2.1, C_U8_1.2, C_U8_2.2, C_VIS_OUT.1, J_CAM.10 (Pin_10), J_CAM.11 (Pin_11), J_CAM.4 (Pin_4), J_CAM.6 (Pin_6), R_CAM_SCL.1, R_CAM_SDA.1, R_VIS_BOOT.1, R_VIS_EN.1, U8.2 (3V3), U_LDO_VIS.2 (VO)
- new net +5V_TOF: C_TOF_OUT.1, D_CAM_LED.2 (A), J_CAM_LED.1 (Pin_1), J_TOF.1 (Pin_1), U_REG_5V_TOF.2 (VO)
- new net BOOT_VIS: R_VIS_BOOT.2, SW_VIS_BOOT.2, U8.27 (IO0)
- new net CAM_D0: J_CAM.19 (Pin_19), U8.19 (IO11)
- new net CAM_D1: J_CAM.21 (Pin_21), U8.17 (IO9)
- new net CAM_D2: J_CAM.22 (Pin_22), U8.12 (IO8)
- new net CAM_D3: J_CAM.20 (Pin_20), U8.18 (IO10)
- new net CAM_D4: J_CAM.18 (Pin_18), U8.20 (IO12)
- new net CAM_D5: J_CAM.16 (Pin_16), U8.11 (IO18)
- new net CAM_D6: J_CAM.14 (Pin_14), U8.10 (IO17)
- new net CAM_D7: J_CAM.12 (Pin_12), U8.9 (IO16)
- new net CAM_HREF: J_CAM.9 (Pin_9), U8.7 (IO7)
- new net CAM_LED_DRAIN: D_CAM_LED.1 (K), J_CAM_LED.2 (Pin_2), Q_CAM_LED.3 (D)
- new net CAM_LED_PWM: R_CAM_LED.1, U8.15 (IO3)
- new net CAM_PCLK: J_CAM.17 (Pin_17), U8.21 (IO13)
- new net CAM_PWDN: J_CAM.8 (Pin_8), U8.24 (IO47)
- new net CAM_SCL: J_CAM.5 (Pin_5), R_CAM_SCL.2, U8.5 (IO5)
- new net CAM_SDA: J_CAM.3 (Pin_3), R_CAM_SDA.2, U8.4 (IO4)
- new net CAM_VSYNC: J_CAM.7 (Pin_7), U8.6 (IO6)
- new net CAM_XCLK: J_CAM.13 (Pin_13), U8.8 (IO15)
- new net TOF_RXD: J_TOF.3 (Pin_3), U8.39 (IO1)
- new net TOF_TXD: J_TOF.4 (Pin_4), U8.38 (IO2)
- new net VBUS_MAIN: C_VBUS_MAIN.2, J2.A4 (VBUS), J2.A9 (VBUS), J2.B4 (VBUS), J2.B9 (VBUS)
- new net VBUS_VIS: C_VBUS_VIS.2, J3.A4 (VBUS), J3.A9 (VBUS), J3.B4 (VBUS), J3.B9 (VBUS)
- new net VIS_USB_D+: J3.A6 (D+), J3.B6 (D+), U8.14 (USB_D+)
- new net VIS_USB_D-: J3.A7 (D-), J3.B7 (D-), U8.13 (USB_D-)
- no-connect marks 48 -> 60
Other:
- note added: "Dual AMS1117 LDOs, OV3660 DVP Camera, MaixSense ToF Sensor, LED Spotlight Driver, Dual Type-C Ports"
- note added: "SECTION 9: ESP32-S3 VISION COPROCESSOR & TRIPLE USB-C INTERFACE"

Commit message: servo pwm alignments. repo & schematic cleanup
Parts:
- removed J_BAT: 2S_LiPo_7.4V, Connector_AMASS:AMASS_XT30PW-M_1x02_P2.50mm_Horizontal, symbol Connector_Generic:Conn_01x02
- removed J_SW_EXT: SW_EXT, Connector_PinHeader_2.54mm:PinHeader_1x02_P2.54mm_Vertical, symbol Connector_Generic:Conn_01x02
- removed R_3V3_LED: 1k, Resistor_SMD:R_0603_1608Metric, symbol Device:R
- removed SW_PWR: POWER_SWITCH, Button_Switch_THT:SW_Slide_SPDT_Straight_CK_OS102011MS2Q, symbol Connector_Generic:Conn_01x03
- added J_BAT1: 2S_LiPo_7.4V, Connector_AMASS:AMASS_XT30PW-M_1x02_P2.50mm_Horizontal, symbol Connector_Generic:Conn_01x02
- added J_SW_EXT1: EXT_SW, Connector_PinHeader_2.54mm:PinHeader_1x02_P2.54mm_Vertical, symbol Connector_Generic:Conn_01x02
- added R_3V3_LED1: 1k, Resistor_SMD:R_0603_1608Metric, symbol Device:R
- added SW_PWR1: PWR_SW, Button_Switch_THT:SW_Slide_SPDT_Straight_CK_OS102011MS2Q, symbol Connector_Generic:Conn_01x03
- added U3: BQ25887RGE, Package_DFN_QFN:Texas_RGE0024H_VQFN-24-1EP_4x4mm_P0.5mm_EP2.7x2.7mm_ThermalVias, symbol Battery_Management:BQ25887RGE
- J_AUX1: value AUX_PWM_18 -> AUX_R_9
- J_AUX2: value AUX_PWM_19 -> AUX_R_10
- J_AUX3: value AUX_PWM_20 -> AUX_R_11
- J_AUX4: value AUX_PWM_21 -> AUX_L_9
- J_AUX5: value AUX_PWM_22 -> AUX_L_10
- J_AUX6: value AUX_PWM_23 -> AUX_L_11
- J_L1_C1: renamed from J_L1_C; value L1_Coxa -> RF_Coxa
- J_L1_F1: renamed from J_L1_F; value L1_Femur -> RF_Femur
- J_L1_T1: renamed from J_L1_T; value L1_Tibia -> RF_Tibia
- J_L2_C1: renamed from J_L2_C; value L2_Coxa -> RM_Coxa
- J_L2_F1: renamed from J_L2_F; value L2_Femur -> RM_Femur
- J_L2_T1: renamed from J_L2_T; value L2_Tibia -> RM_Tibia
- J_L3_C1: renamed from J_L3_C; value L3_Coxa -> RR_Coxa
- J_L3_F1: renamed from J_L3_F; value L3_Femur -> RR_Femur
- J_L3_T1: renamed from J_L3_T; value L3_Tibia -> RR_Tibia
- J_L4_C1: renamed from J_L4_C; value L4_Coxa -> LF_Coxa
- J_L4_F1: renamed from J_L4_F; value L4_Femur -> LF_Femur
- J_L4_T1: renamed from J_L4_T; value L4_Tibia -> LF_Tibia
- J_L5_C1: renamed from J_L5_C; value L5_Coxa -> LM_Coxa
- J_L5_F1: renamed from J_L5_F; value L5_Femur -> LM_Femur
- J_L5_T1: renamed from J_L5_T; value L5_Tibia -> LM_Tibia
- J_L6_C1: renamed from J_L6_C; value L6_Coxa -> LR_Coxa
- J_L6_F1: renamed from J_L6_F; value L6_Femur -> LR_Femur
- J_L6_T1: renamed from J_L6_T; value L6_Tibia -> LR_Tibia
- renumbered C_DIV to C_DIV1, C_IN1_L to C_IN1_L1, C_IN1_R to C_IN1_R1, C_IN2_L to C_IN2_L1, C_IN2_R to C_IN2_R1, C_NEO to C_NEO1, C_OUT1_L to C_OUT1_L1, C_OUT1_R to C_OUT1_R1, C_OUT2_L to C_OUT2_L1, C_OUT2_R to C_OUT2_R1, C_OUT3_L to C_OUT3_L1, C_OUT3_R to C_OUT3_R1, C_TOF_IN to C_TOF_IN1, C_TOF_OUT to C_TOF_OUT1, C_VBUS_MAIN to C_VBUS_MAIN1, C_VBUS_VIS to C_VBUS_VIS1, C_VIS_EN to C_VIS_EN1, C_VIS_IN to C_VIS_IN1, C_VIS_OUT to C_VIS_OUT1, D_CAM_LED to D_CAM_LED1, D_CATCH_L to D_CATCH_L1, D_CATCH_R to D_CATCH_R1, D_ISO to D_ISO1, D_STAT to D_STAT1, J_CAM to J_CAM1, J_CAM_LED to J_CAM_LED1, J_I2C to J_I2C1, J_TOF to J_TOF1, J_UART to J_UART1, LED_CHG to LED_CHG1, LED_FULL to LED_FULL1, LED_L to LED_L1, LED_R to LED_R1, LED_RGB_MAIN to LED_RGB_MAIN1, L_CHG to L_CHG1, L_SERVO_L to L_SERVO_L1, L_SERVO_R to L_SERVO_R1, Q_CAM_LED to Q_CAM_LED1, R_BZ to R_BZ1, R_CAM_LED to R_CAM_LED1, R_CAM_SCL to R_CAM_SCL1, R_CAM_SDA to R_CAM_SDA1, R_CHG to R_CHG1, R_FB1_L to R_FB1_L1, R_FB1_R to R_FB1_R1, R_FB2_L to R_FB2_L1, R_FB2_R to R_FB2_R1, R_FULL to R_FULL1, R_LED_L to R_LED_L1, R_LED_R to R_LED_R1, R_NEO to R_NEO1, R_OE to R_OE1, R_PD_CAM_LED to R_PD_CAM_LED1, R_SCL to R_SCL1, R_SDA to R_SDA1, R_STAT to R_STAT1, R_VIS_BOOT to R_VIS_BOOT1, R_VIS_EN to R_VIS_EN1, SW_VIS_BOOT to SW_VIS_BOOT1, SW_VIS_RST to SW_VIS_RST1, U3_L to U3_L1, U3_R to U3_R1, U_LDO_VIS to U_LDO_VIS1, U_REG_5V_TOF to U_REG_5V_TOF1
Connections:
- net GND: now also J_BAT1.2 (Pin_2), R_3V3_LED1.2; no longer LED_3V3.2 (A)
- net VBAT: now also J_BAT1.1 (Pin_1), J_SW_EXT1.1 (Pin_1), SW_PWR1.1 (Pin_1)
- net VBAT_SW: now also J_SW_EXT1.2 (Pin_2), SW_PWR1.2 (Pin_2), SW_PWR1.3 (Pin_3)
- net V_SERVO_L: now also R_FB1_L1.2; no longer R_FB1_L1.1
- net V_SERVO_R: now also R_FB1_R1.2; no longer R_FB1_R1.1
- net PWM_L_8: now reaches U6.15 (LED8)
- net PWM_L_8: now also J_L6_T1.3 (Pin_3)
- net PWM_L_9: now reaches U6.16 (LED9)
- net PWM_L_9: now also J_AUX4.3 (Pin_3)
- net PWM_L_10: now reaches U6.17 (LED10)
- net PWM_L_10: now also J_AUX5.3 (Pin_3)
- net PWM_L_11: now reaches U6.18 (LED11)
- net PWM_L_11: now also J_AUX6.3 (Pin_3)
- net BUCK_FB_L: no longer names the net of R_FB2_L1.1, U3_L1.2 (FB)
- net BUCK_FB_L: now also R_FB1_L1.1; no longer R_FB1_L1.2
- net BUCK_FB_R: no longer names the net of R_FB2_R1.1, U3_R1.2 (FB)
- net BUCK_FB_R: now also R_FB1_R1.1; no longer R_FB1_R1.2
- net BUCK_SW_L: no longer names the net of D_CATCH_L1.2 (A), L_SERVO_L1.1, U3_L1.3 (SW)
- net BUCK_SW_R: no longer names the net of D_CATCH_R1.2 (A), L_SERVO_R1.1, U3_R1.3 (SW)
- net PWM_0 renamed PWM_R_0
- net PWM_1 renamed PWM_R_1
- net PWM_10 renamed PWM_L_1
- net PWM_L_1: now also U6.7 (LED1); no longer U5.17 (LED10)
- net PWM_11 renamed PWM_L_2
- net PWM_L_2: now also U6.8 (LED2); no longer U5.18 (LED11)
- net PWM_12: no longer names the net of U5.19 (LED12)
- net PWM_12: no longer J_L5_C1.3 (Pin_3)
- net PWM_13: no longer names the net of U5.20 (LED13)
- net PWM_13: no longer J_L5_F1.3 (Pin_3)
- net PWM_14: no longer names the net of U5.21 (LED14)
- net PWM_14: no longer J_L5_T1.3 (Pin_3)
- net PWM_15: no longer names the net of U5.22 (LED15)
- net PWM_15: no longer J_L6_C1.3 (Pin_3)
- net PWM_16 renamed PWM_L_0
- net PWM_L_0: now also J_L4_C1.3 (Pin_3); no longer J_L6_F1.3 (Pin_3)
- removed net PWM_17: J_L6_T1.3 (Pin_3), U6.7 (LED1)
- net PWM_18 renamed PWM_R_9
- net PWM_R_9: now also U5.16 (LED9); no longer U6.8 (LED2)
- net PWM_19 renamed PWM_L_3
- net PWM_L_3: now also J_L5_C1.3 (Pin_3); no longer J_AUX2.3 (Pin_3)
- net PWM_2 renamed PWM_R_2
- net PWM_20 renamed PWM_L_4
- net PWM_L_4: now also J_L5_F1.3 (Pin_3); no longer J_AUX3.3 (Pin_3)
- net PWM_21 renamed PWM_L_5
- net PWM_L_5: now also J_L5_T1.3 (Pin_3); no longer J_AUX4.3 (Pin_3)
- net PWM_22 renamed PWM_L_6
- net PWM_L_6: now also J_L6_C1.3 (Pin_3); no longer J_AUX5.3 (Pin_3)
- net PWM_23 renamed PWM_L_7
- net PWM_L_7: now also J_L6_F1.3 (Pin_3); no longer J_AUX6.3 (Pin_3)
- net PWM_3 renamed PWM_R_3
- net PWM_4 renamed PWM_R_4
- net PWM_5 renamed PWM_R_5
- net PWM_6 renamed PWM_R_6
- net PWM_7 renamed PWM_R_7
- net PWM_8 renamed PWM_R_8
- removed net PWM_9: J_L4_C1.3 (Pin_3), U5.16 (LED9)
- new net: U3.13 (BAT), U3.14 (BAT)
- new net: U3.15 (SNS), U3.16 (SNS)
- new net: U3.17 (SW), U3.18 (SW)
- new net: U3.19 (GND), U3.20 (GND), U3.25 (GND)
- new net: U3.21 (PMID), U3.22 (PMID)
- new net: LED_3V3.2 (A), R_3V3_LED1.1
- new net PWM_R_10: J_AUX2.3 (Pin_3), U5.17 (LED10)
- new net PWM_R_11: J_AUX3.3 (Pin_3), U5.18 (LED11)
Other:
- note added: "SECTION 8: MPU-6050 6-DOF IMU"
- note removed: "SECTION 8: MPU-6050 6-AXIS MOTION TRACKING SENSOR"
- moved on the sheet: C_BAT1, C_BAT2, C_MPU1, C_MPU3, C_PCA1, C_PCA2, C_PCA3, C_PCA4, C_VBUS1, C_VBUS2, D_ISO1, J1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
